Commit message: finish week2 assignments

File: hrwros_week2/urdf/hrwros_assignment1.xacro (robot description, xacro)
@@ -72,3 +72,10 @@
   </joint>
   <!-- Add your solution to assignment 1 here -->
+  <xacro:bin_urdf prefix="bin_2_"/>
+  <!-- bin 1 -->
+  <joint name="bin_2_joint" type="fixed">
+    <parent link="world_interface" />
+    <child link="bin_2_base_link" />
+    <origin xyz="2.5 1.8 0" rpy="0 0 0" />
+  </joint>
 </robot>

File: hrwros_week2/urdf/hrwros_assignment2.xacro (robot description, xacro)
@@ -72,3 +72,20 @@
   </joint>
   <!-- Add your solution to assignment 2 here -->
+  <link name="sphere_link">
+    <visual>
+      <origin xyz="0 0 0" />
+      <geometry>
+        <sphere radius ="0.4"/>
+      </geometry>
+      <material name="green">
+        <color rgba="0 0.9 0 1"/>
+      </material>
+    </visual>
+  </link>
+  <!-- Add your solution to assignment 2 here -->
+  <joint name="sphere_joint" type="fixed">
+    <origin xyz="5.8 -5.3 0" />
+    <parent link="world" />
+    <child link="sphere_link" />
+  </joint>
 </robot>

File: hrwros_week2/urdf/hrwros_assignment3.xacro (robot description, xacro)
@@ -65,10 +65,10 @@
   </joint>
   <!-- Update the below block for assignment 3 here -->
-  <xacro:include filename="$(find ur_description)/urdf/ur5.urdf.xacro"/>
-  <xacro:ur5_robot prefix="robot2_" joint_limited="true"/>
+  <xacro:include filename="$(find hrwros_week2)/urdf/robot/lrmate200ic_macro.xacro"/>
+  <xacro:fanuc_lrmate200ic prefix="robot2_" joint_limited="true"/>
   <joint name="robot2-robot2_pedestal_joint" type="fixed">
     <parent link="robot2_pedestal_link" />
     <child link="robot2_base_link" />
-    <origin xyz="0 0 0.6" rpy="0 0 ${radians(90)}" />
+    <origin xyz="0 0 0.6" rpy="0 0 ${radians(180)}" />
   </joint>
 </robot>
