Commit message: fix week2 assignment mistake

File: hrwros_week2/urdf/hrwros_assignment2.xacro (robot description, xacro)
@@ -85,5 +85,5 @@
   <!-- Add your solution to assignment 2 here -->
   <joint name="sphere_joint" type="fixed">
-    <origin xyz="5.8 -5.3 0" />
+    <origin xyz="5.8 -5.3 0.4" />
     <parent link="world" />
     <child link="sphere_link" />
