Commit message: finish week6 assignment

File: hrwros_support/urdf/break_beam/break_beam.gazebo.xacro (robot description, xacro)
@@ -22,5 +22,5 @@
           <range>
             <min>0.10</min>
-            <max>1.0</max>
+            <max>0.6</max>
             <resolution>0.01</resolution>
           </range>

File: hrwros_support/urdf/break_beam/break_beam.urdf.xacro (robot description, xacro)
@@ -34,5 +34,5 @@
       <parent link="${prefix}world_interface" />
       <child link="${prefix}base_link" />
-      <origin xyz="1.6 2.7 0.925" rpy="0 0 ${radians(180)}" />
+      <origin xyz="1.6 1.9 0.925" rpy="0 0 ${radians(180)}" />
     </joint>
     <joint name="${prefix}joint_1" type="fixed">

File: hrwros_support/urdf/hrwros.xacro (robot description, xacro)
@@ -31,7 +31,7 @@
   <xacro:include filename="$(find hrwros_support)/urdf/bin/bin.urdf.xacro"/>
   <xacro:bin_urdf prefix="bin_1_"/>
-  <!-- depth camera -->
-  <xacro:include filename="$(find hrwros_support)/urdf/depth_camera/depth_camera.urdf.xacro"/>
-  <xacro:depth_camera_urdf prefix="depth_camera_"/>
+  <!-- logical camera collision model -->
+  <xacro:include filename="$(find hrwros_support)/urdf/logical_camera/logical_camera.urdf.xacro"/>
+  <xacro:logical_camera_urdf prefix="logical_camera1_"/>
   <!-- break beam -->
   <xacro:include filename="$(find hrwros_support)/urdf/break_beam/break_beam.urdf.xacro"/>
@@ -50,6 +50,6 @@
   <!-- robot1 to pedestal. -->
   <joint name="robot1_to_pedestal" type="fixed">
-  <origin xyz="0 0 0.95" rpy="0 0 0" />
-  <parent link="robot1_pedestal_link" />
+  <origin xyz="0.5 1.8 0.95" rpy="0 0 0" />
+  <parent link="world_interface" />
   <child link="robot1_base_link" />
   </joint>
@@ -67,7 +67,7 @@
   <!-- robot2 to pedestal. -->
   <joint name="robot2_to_pedestal" type="fixed">
-    <parent link="robot2_pedestal_link" />
+    <parent link="world_interface" />
     <child link="robot2_base_link" />
-    <origin xyz="0 0 0.7" rpy="0 0 ${radians(90)}" />
+    <origin xyz="-7.8 -1.5 0.7" rpy="0 0 ${radians(90)}" />
   </joint>
   <!-- gripper2 to robot2. -->
@@ -81,9 +81,4 @@
     <child link="break_beam_world_interface" />
   </joint>
-  <!-- TODO: Replace this with logical camera. -->
-  <joint name="camera_link" type="fixed">
-    <parent link="world_interface"/>
-    <child link="depth_camera_world_interface" />
-  </joint>
   <!-- bin to world. -->
   <joint name="bin_1_joint" type="fixed">
@@ -92,3 +87,8 @@
     <origin xyz="-8.0 -2.2 0.0" rpy="0 0 0" />
   </joint>
+  <!-- logicam1 to world. -->
+  <joint name="logicam_world_interface" type="fixed">
+    <parent link="world_interface" />
+    <child link="logical_camera1_world_interface" />
+  </joint>
 </robot>

File: hrwros_support/urdf/robot_system/robot_system.gazebo.xacro (robot description, xacro)
@@ -1,5 +1,18 @@
 <?xml version="1.0"?>
 <robot name="robot_system" xmlns:xacro="http://www.ros.org/wiki/xacro">
-  <xacro:macro name="robot_system_gazebo" params="robot_prefix robot_parameter_name">
+  <xacro:macro name="robot_system_gazebo" params="robot_prefix robot_parameter_name vacuum_gripper_prefix gripper_plugin_name">
+    <!-- Vacuum Gripper -->
+    <xacro:if value="${robot_prefix == 'robot1_'}">
+      <xacro:include filename="$(find hrwros_support)/urdf/vacuum_gripper/vacuum_gripper.gazebo.xacro"/>
+      <xacro:vacuum_gripper_gazebo prefix="${vacuum_gripper_prefix}" gripper_link="robot1::${robot_prefix}wrist_3_link" plugin_name = "${gripper_plugin_name}">
+        <drops_info/>
+      </xacro:vacuum_gripper_gazebo>
+    </xacro:if>
+    <xacro:if value="${robot_prefix == 'robot2_'}">
+      <xacro:include filename="$(find hrwros_support)/urdf/vacuum_gripper/vacuum_gripper.gazebo.xacro"/>
+      <xacro:vacuum_gripper_gazebo prefix="${vacuum_gripper_prefix}" gripper_link="robot2::${robot_prefix}wrist_3_link" plugin_name = "${gripper_plugin_name}">
+        <drops_info/>
+      </xacro:vacuum_gripper_gazebo>
+    </xacro:if>
     <gazebo reference="${robot_prefix}base_link">
       <turnGravityOff>true</turnGravityOff>
@@ -26,4 +39,7 @@
       <turnGravityOff>true</turnGravityOff>
     </gazebo>
+    <gazebo reference="${vacuum_gripper_prefix}suction_cup">
+      <turnGravityOff>true</turnGravityOff>
+    </gazebo>
     <gazebo>
       <plugin name="gazebo_ros_control" filename="libgazebo_ros_control.so">

File: hrwros_support/urdf/robot_system/robot_system.xacro (robot description, xacro)
@@ -5,9 +5,10 @@
   <xacro:arg name="vacuum_gripper_prefix" default="vacuum_gripper1_"/>
   <xacro:arg name="robot_param" default="/robot1/robot1_description"/>
+   <xacro:arg name="gripper_plugin_name" default="gripper1"/>
   <!-- URDF -->
   <xacro:include filename="$(find hrwros_support)/urdf/robot_system/robot_system.urdf.xacro"/>
-  <xacro:robot_system_urdf robot_type= "$(arg robot_type)" robot_prefix="$(arg robot_prefix)" vacuum_gripper_prefix="$(arg vacuum_gripper_prefix"/>
+  <xacro:robot_system_urdf robot_type= "$(arg robot_type)" robot_prefix="$(arg robot_prefix)" vacuum_gripper_prefix="$(arg vacuum_gripper_prefix)"/>
   <!-- Gazebo -->
   <xacro:include filename="$(find hrwros_support)/urdf/robot_system/robot_system.gazebo.xacro"/>
-  <xacro:robot_system_gazebo robot_prefix="$(arg robot_prefix)" robot_parameter_name="$(arg robot_param)"/>
+  <xacro:robot_system_gazebo robot_prefix="$(arg robot_prefix)" robot_parameter_name="$(arg robot_param)" vacuum_gripper_prefix="$(arg vacuum_gripper_prefix)" gripper_plugin_name="$(arg gripper_plugin_name)"/>
 </robot>

File: hrwros_support/urdf/vacuum_gripper/vacuum_gripper.urdf.xacro (robot description, xacro)
@@ -22,14 +22,38 @@
       <inertial>
         <origin xyz="0 0 0" rpy="0 0 0" />
-        <inertia ixx="0.00001" ixy="0" ixz="0"
-                 iyy="0.00001" iyz="0"
-                 izz="0.00001" />
+        <inertia ixx="1.0" ixy="0" ixz="0"
+                 iyy="1.0" iyz="0"
+                 izz="1.0" />
+        <mass value="1.0" />
+      </inertial>
+    </link>
+    <link name="${prefix}suction_cup">
+      <visual>
+        <origin xyz="0 0 0" rpy="0 0 0" />
+        <geometry>
+          <box size="0.001 0.001 0.001" />
+        </geometry>
+        <material name="red">
+          <color rgba="1 0 0 1"/>
+        </material>
+      </visual>
+      <collision>
+        <origin xyz="0 0 0" rpy="0 0 0"/>
+        <geometry>
+          <box size="0.001 0.001 0.001" />
+        </geometry>
+        <material name="red"/>
+      </collision>
+      <inertial>
+        <origin xyz="0 0 0" rpy="0 0 0" />
+        <inertia ixx="0.0001" ixy="0" ixz="0"
+                 iyy="0.0001" iyz="0"
+                 izz="0.0001" />
         <mass value="0.00001" />
       </inertial>
     </link>
-    <link name="${prefix}suction_cup"/>
     <!-- joint list -->
     <joint name="${joint_prefix}" type="fixed">
-      <origin xyz="0 0 0.080" rpy="0 0 0" />
+      <origin xyz="0 0 0.01" rpy="0 0 0" />
       <parent link="${prefix}base_link" />
       <child link="${prefix}suction_cup" />
